Commit message: [urdf] trunk_large visual correctly match collision shape

File: data/talos/urdf/talos_trunk_large.urdf (robot description, URDF)
Before this commit: robot talos_trunk, 3 links, 2 joints
Links:
- link base_link: geometry collision mesh filename=package://talos-rbprm/meshes/talos_trunk_lower_large.stl scale=1 1 1; visual mesh filename=package://talos-rbprm/meshes/talos_trunk_lower_visual_large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 scale=1 1 1
